Commit message: Beginning to add wheels. Model Builds

File: urdf/robot.xacro (robot description, xacro)
@@ -9,4 +9,10 @@
   <!-- <xacro:include filename="$(find enph353_ros_lab)/urdf/robot.gazebo" /> -->
   <xacro:include filename="$(find enph353_ros_lab)/urdf/macros.xacro" />
+  <material name="blue">
+    <color rgba="0 0 0.8 1"/>
+  </material>
+  <material name="black">
+    <color rgba="0 0 0 1"/>
+  </material>
   <link name='chassis'>
     <xacro:box_inertial name="chassis" m="${chassis_mass}" x="${chassis_length}" y="${chassis_width}" z="${chassis_height}"/>
@@ -16,4 +22,5 @@
       </geometry>
     </collision>
+    <xacro:default_inertial mass="1"/>
     <visual name='chassis_visual'>
       <origin xyz="0 0 0" rpy=" 0 0 0"/>
@@ -23,3 +30,37 @@
     </visual>
   </link>
+  <link name="right_front_wheel">
+    <visual>
+      <origin rpy="1.57075 0 0" xyz="0 0 0"/>
+      <geometry>
+        <cylinder length="${wheel_width}" radius="${wheel_radius}"/>
+      </geometry>
+      <material name="black"/>
+      <origin rpy="0 0 0" xyz="0 0 0"/>
+    </visual>
+    <collision name='chassis_collision'>
+      <geometry>
+        <cylinder length="${wheel_width}" radius="${wheel_radius}"/>
+      </geometry>
+    </collision>
+  </link>
+  <joint name="right_front_wheel_joint" type="fixed">
+    <parent link="chassis"/>
+    <child link="right_front_wheel"/>
+    <origin rpy="0 0 0" xyz="0.133333333333 0 -0.085"/>
+  </joint>
+  <!-- <link name="right_back_wheel">
+    <visual>
+      <origin rpy="1.57075 0 0" xyz="0 0 0"/>
+      <geometry>
+        <cylinder length="0.1" radius="0.035"/>
+      </geometry>
+      <material name="black"/>
+    </visual>
+  </link>
+  <joint name="right_back_wheel_joint" type="fixed">
+    <parent link="chassis"/>
+    <child link="right_back_wheel"/>
+    <origin rpy="0 0 0" xyz="-0.133333333333 0 -0.085"/>
+  </joint> -->
 </robot>

Commit message: fixed inntertia

File: urdf/robot.xacro (robot description, xacro)
@@ -9,4 +9,10 @@
   <!-- <xacro:include filename="$(find enph353_ros_lab)/urdf/robot.gazebo" /> -->
   <xacro:include filename="$(find enph353_ros_lab)/urdf/macros.xacro" />
+  <xacro:macro name="default_inertial" params="mass">
+    <inertial>
+      <mass value="${mass}" />
+      <inertia ixx="1.0" ixy="0.0" ixz="0.0" iyy="1.0" iyz="0.0" izz="1.0" />
+    </inertial>
+  </xacro:macro>
   <material name="blue">
     <color rgba="0 0 0.8 1"/>

Commit message: Wheel with continuous joint

File: urdf/robot.xacro (robot description, xacro)
@@ -37,4 +37,5 @@
   </link>
   <link name="right_front_wheel">
+    <xacro:default_inertial mass="0.1"/>
     <visual>
       <origin rpy="1.57075 0 0" xyz="0 0 0"/>
@@ -45,5 +46,5 @@
       <origin rpy="0 0 0" xyz="0 0 0"/>
     </visual>
-    <collision name='chassis_collision'>
+    <collision name='wheel_collision'>
       <geometry>
         <cylinder length="${wheel_width}" radius="${wheel_radius}"/>
@@ -51,8 +52,9 @@
     </collision>
   </link>
-  <joint name="right_front_wheel_joint" type="fixed">
+  <joint name="right_front_wheel_joint" type="continuous">
+    <axis xyz="0 1 0" />
     <parent link="chassis"/>
     <child link="right_front_wheel"/>
-    <origin rpy="0 0 0" xyz="0.133333333333 0 -0.085"/>
+    <origin rpy="0 0 0" xyz="0 0 0"/>
   </joint>
   <!-- <link name="right_back_wheel">

Commit message: camera works

File: urdf/robot.xacro (robot description, xacro)
@@ -7,4 +7,5 @@
   <xacro:property name="wheel_radius" value="0.04"/>
   <xacro:property name="wheel_width" value="0.03"/>
+  <xacro:property name="camera_link" value="0.05" />
   <!-- <xacro:include filename="$(find enph353_ros_lab)/urdf/robot.gazebo" /> -->
   <xacro:include filename="$(find enph353_ros_lab)/urdf/macros.xacro" />
@@ -56,4 +57,71 @@
     <origin rpy="0 0 0" xyz="0.133333333333 0 -0.085"/>
   </joint>
+ <!-- Camera -->
+ <joint name="camera_joint" type="fixed">
+    <axis xyz="0 1 0" />
+    <origin xyz="0 0 0" rpy="0 0 0"/>
+    <parent link="chassis"/>
+    <child link="camera_link"/>
+  </joint>
+  <xacro:property name="camera_link" value="0.05" /> <!-- Size of square 'camera' box -->
+  <link name="camera_link">
+    <collision>
+      <origin xyz="0 0 0" rpy="0 0 0"/>
+      <geometry>
+    <box size="${camera_link} ${camera_link} ${camera_link}"/>
+      </geometry>
+    </collision>
+    <visual>
+      <origin xyz="0 0 0" rpy="0 0 0"/>
+      <geometry>
+    <box size="${camera_link} ${camera_link} ${camera_link}"/>
+      </geometry>
+      <material name="red"/>
+    </visual>
+    <inertial>
+      <mass value="1e-5" />
+      <origin xyz="0 0 0" rpy="0 0 0"/>
+      <inertia ixx="1e-6" ixy="0" ixz="0" iyy="1e-6" iyz="0" izz="1e-6" />
+    </inertial>
+  </link>
+<gazebo reference="camera_link">
+    <sensor type="camera" name="camera1">
+      <update_rate>30.0</update_rate>
+      <camera name="head">
+        <horizontal_fov>1.3962634</horizontal_fov>
+        <image>
+          <width>800</width>
+          <height>800</height>
+          <format>R8G8B8</format>
+        </image>
+        <clip>
+          <near>0.02</near>
+          <far>300</far>
+        </clip>
+        <noise>
+          <type>gaussian</type>
+          <!-- Noise is sampled independently per pixel on each frame.
+               That pixel's noise value is added to each of its color
+               channels, which at that point lie in the range [0,1]. -->
+          <mean>0.0</mean>
+          <stddev>0.007</stddev>
+        </noise>
+      </camera>
+      <plugin name="camera_controller" filename="libgazebo_ros_camera.so">
+        <alwaysOn>true</alwaysOn>
+        <updateRate>0.0</updateRate>
+        <cameraName>rrbot/camera1</cameraName>
+        <imageTopicName>image_raw</imageTopicName>
+        <cameraInfoTopicName>camera_info</cameraInfoTopicName>
+        <frameName>camera_link</frameName>
+        <hackBaseline>0.07</hackBaseline>
+        <distortionK1>0.0</distortionK1>
+        <distortionK2>0.0</distortionK2>
+        <distortionK3>0.0</distortionK3>
+        <distortionT1>0.0</distortionT1>
+        <distortionT2>0.0</distortionT2>
+      </plugin>
+    </sensor>
+  </gazebo>
   <!-- <link name="right_back_wheel">
     <visual>

Commit message: cleaned up double declaration

File: urdf/robot.xacro (robot description, xacro)
@@ -64,5 +64,4 @@
     <child link="camera_link"/>
   </joint>
-  <xacro:property name="camera_link" value="0.05" /> <!-- Size of square 'camera' box -->
   <link name="camera_link">
     <collision>

Commit message: Back wheels don't work

File: urdf/robot.xacro (robot description, xacro)
@@ -36,4 +36,26 @@
     </visual>
   </link>
+  <link name="left_front_wheel">
+    <xacro:default_inertial mass="0.1"/>
+    <visual>
+      <origin rpy="1.57075 0 0" xyz="0 0 0"/>
+      <geometry>
+        <cylinder length="${wheel_width}" radius="${wheel_radius}"/>
+      </geometry>
+      <material name="black"/>
+      <origin rpy="0 0 0" xyz="0 0 0"/>
+    </visual>
+    <collision name='wheel_collision'>
+      <geometry>
+        <cylinder length="${wheel_width}" radius="${wheel_radius}"/>
+      </geometry>
+    </collision>
+  </link>
+  <joint name="left_front_wheel_joint" type="continuous">
+    <axis xyz="0 1 0" />
+    <parent link="chassis"/>
+    <child link="left_front_wheel"/>
+    <origin rpy="0 0 0" xyz="0.1 0.075 0"/>
+  </joint>
   <link name="right_front_wheel">
     <xacro:default_inertial mass="0.1"/>
@@ -56,19 +78,49 @@
     <parent link="chassis"/>
     <child link="right_front_wheel"/>
-    <origin rpy="0 0 0" xyz="0 0 0"/>
+    <origin rpy="0 0 0" xyz="0.1 -0.075 0"/>
   </joint>
-  <!-- <link name="right_back_wheel">
+  <!-- <link name="left_back_wheel">
+    <xacro:default_inertial mass="0.1"/>
     <visual>
       <origin rpy="1.57075 0 0" xyz="0 0 0"/>
       <geometry>
-        <cylinder length="0.1" radius="0.035"/>
+        <cylinder length="${wheel_width}" radius="${wheel_radius}"/>
       </geometry>
       <material name="black"/>
+      <origin rpy="0 0 0" xyz="0 0 0"/>
     </visual>
+    <collision name='wheel_collision'>
+      <geometry>
+        <cylinder length="${wheel_width}" radius="${wheel_radius}"/>
+      </geometry>
+    </collision>
   </link>
-  <joint name="right_back_wheel_joint" type="fixed">
+  <joint name="left_back_wheel_joint" type="continuous">
+    <axis xyz="0 1 0" />
+    <parent link="chassis"/>
+    <child link="left_back_wheel"/>
+    <origin rpy="0 0 0" xyz="-0.1 0.075 0"/>
+  </joint> -->
+  <!-- <link name="right_back_wheel">
+    <xacro:default_inertial mass="0.1"/>
+    <visual>
+      <origin rpy="1.57075 0 0" xyz="0 0 0"/>
+      <geometry>
+        <cylinder length="${wheel_width}" radius="${wheel_radius}"/>
+      </geometry>
+      <material name="black"/>
+      <origin rpy="0 0 0" xyz="0 0 0"/>
+    </visual>
+    <collision name='wheel_collision'>
+      <geometry>
+        <cylinder length="${wheel_width}" radius="${wheel_radius}"/>
+      </geometry>
+    </collision>
+  </link>
+  <joint name="right_back_wheel_joint" type="continuous">
+    <axis xyz="0 1 0" />
     <parent link="chassis"/>
     <child link="right_back_wheel"/>
-    <origin rpy="0 0 0" xyz="-0.133333333333 0 -0.085"/>
+    <origin rpy="0 0 0" xyz="-0.1 -0.08 0"/>
   </joint> -->
 </robot>

Commit message: YESSS Built a car with 4 wheels

File: urdf/robot.xacro (robot description, xacro)
@@ -37,17 +37,17 @@
   </link>
   <link name="left_front_wheel">
-    <xacro:default_inertial mass="0.1"/>
-    <visual>
-      <origin rpy="1.57075 0 0" xyz="0 0 0"/>
-      <geometry>
-        <cylinder length="${wheel_width}" radius="${wheel_radius}"/>
-      </geometry>
-      <material name="black"/>
-      <origin rpy="0 0 0" xyz="0 0 0"/>
-    </visual>
-    <collision name='wheel_collision'>
-      <geometry>
-        <cylinder length="${wheel_width}" radius="${wheel_radius}"/>
-      </geometry>
+    <xacro:cylinder_inertial name="wheel" m="0.1" r="${wheel_radius}" h="${wheel_width}" />
+    <xacro:default_inertial mass="0.1"/>
+    <visual>
+      <origin rpy="1.57075 0 0" xyz="0 0 0"/>
+      <geometry>
+        <cylinder length="${wheel_width}" radius="${wheel_radius}"/>
+      </geometry>>
+    </visual>
+    <collision name='wheel_collision'>
+      <origin rpy="1.57075 0 0" xyz="0 0 0"/>
+      <geometry>
+        <cylinder length="${wheel_width}" radius="${wheel_radius}"/>
+      </geometry>>
     </collision>
   </link>
@@ -56,20 +56,20 @@
     <parent link="chassis"/>
     <child link="left_front_wheel"/>
-    <origin rpy="0 0 0" xyz="0.1 0.075 0"/>
+    <origin rpy="0 0 0" xyz="0.1 0.09 0"/>
   </joint>
   <link name="right_front_wheel">
-    <xacro:default_inertial mass="0.1"/>
-    <visual>
-      <origin rpy="1.57075 0 0" xyz="0 0 0"/>
-      <geometry>
-        <cylinder length="${wheel_width}" radius="${wheel_radius}"/>
-      </geometry>
-      <material name="black"/>
-      <origin rpy="0 0 0" xyz="0 0 0"/>
-    </visual>
-    <collision name='wheel_collision'>
-      <geometry>
-        <cylinder length="${wheel_width}" radius="${wheel_radius}"/>
-      </geometry>
+    <xacro:cylinder_inertial name="wheel" m="0.1" r="${wheel_radius}" h="${wheel_width}" />
+    <xacro:default_inertial mass="0.1"/>
+    <visual>
+      <origin rpy="1.57075 0 0" xyz="0 0 0"/>
+      <geometry>
+        <cylinder length="${wheel_width}" radius="${wheel_radius}"/>
+      </geometry>>
+    </visual>
+    <collision name='wheel_collision'>
+      <origin rpy="1.57075 0 0" xyz="0 0 0"/>
+      <geometry>
+        <cylinder length="${wheel_width}" radius="${wheel_radius}"/>
+      </geometry>>
     </collision>
   </link>
@@ -78,5 +78,49 @@
     <parent link="chassis"/>
     <child link="right_front_wheel"/>
-    <origin rpy="0 0 0" xyz="0.1 -0.075 0"/>
+    <origin rpy="0 0 0" xyz="0.1 -0.09 0"/>
+  </joint>
+  <link name="left_back_wheel">
+    <xacro:cylinder_inertial name="wheel" m="0.1" r="${wheel_radius}" h="${wheel_width}" />
+    <xacro:default_inertial mass="0.1"/>
+    <visual>
+      <origin rpy="1.57075 0 0" xyz="0 0 0"/>
+      <geometry>
+        <cylinder length="${wheel_width}" radius="${wheel_radius}"/>
+      </geometry>>
+    </visual>
+    <collision name='wheel_collision'>
+      <origin rpy="1.57075 0 0" xyz="0 0 0"/>
+      <geometry>
+        <cylinder length="${wheel_width}" radius="${wheel_radius}"/>
+      </geometry>>
+    </collision>
+  </link>
+  <joint name="left_back_wheel_joint" type="continuous">
+    <axis xyz="0 1 0" />
+    <parent link="chassis"/>
+    <child link="left_back_wheel"/>
+    <origin rpy="0 0 0" xyz="-0.1 0.09 0"/>
+  </joint>
+  <link name="right_back_wheel">
+    <xacro:cylinder_inertial name="wheel" m="0.1" r="${wheel_radius}" h="${wheel_width}" />
+    <xacro:default_inertial mass="0.1"/>
+    <visual>
+      <origin rpy="1.57075 0 0" xyz="0 0 0"/>
+      <geometry>
+        <cylinder length="${wheel_width}" radius="${wheel_radius}"/>
+      </geometry>>
+    </visual>
+    <collision name='wheel_collision'>
+      <origin rpy="1.57075 0 0" xyz="0 0 0"/>
+      <geometry>
+        <cylinder length="${wheel_width}" radius="${wheel_radius}"/>
+      </geometry>>
+    </collision>
+  </link>
+  <joint name="right_back_wheel_joint" type="continuous">
+    <axis xyz="0 1 0" />
+    <parent link="chassis"/>
+    <child link="right_back_wheel"/>
+    <origin rpy="0 0 0" xyz="-0.1 -0.09 0"/>
   </joint>
  <!-- Camera -->
@@ -146,48 +190,4 @@
     </sensor>
   </gazebo>
-  <!-- <link name="left_back_wheel">
-    <xacro:default_inertial mass="0.1"/>
-    <visual>
-      <origin rpy="1.57075 0 0" xyz="0 0 0"/>
-      <geometry>
-        <cylinder length="${wheel_width}" radius="${wheel_radius}"/>
-      </geometry>
-      <material name="black"/>
-      <origin rpy="0 0 0" xyz="0 0 0"/>
-    </visual>
-    <collision name='wheel_collision'>
-      <geometry>
-        <cylinder length="${wheel_width}" radius="${wheel_radius}"/>
-      </geometry>
-    </collision>
-  </link>
-  <joint name="left_back_wheel_joint" type="continuous">
-    <axis xyz="0 1 0" />
-    <parent link="chassis"/>
-    <child link="left_back_wheel"/>
-    <origin rpy="0 0 0" xyz="-0.1 0.075 0"/>
-  </joint> -->
-  <!-- <link name="right_back_wheel">
-    <xacro:default_inertial mass="0.1"/>
-    <visual>
-      <origin rpy="1.57075 0 0" xyz="0 0 0"/>
-      <geometry>
-        <cylinder length="${wheel_width}" radius="${wheel_radius}"/>
-      </geometry>
-      <material name="black"/>
-      <origin rpy="0 0 0" xyz="0 0 0"/>
-    </visual>
-    <collision name='wheel_collision'>
-      <geometry>
-        <cylinder length="${wheel_width}" radius="${wheel_radius}"/>
-      </geometry>
-    </collision>
-  </link>
-  <joint name="right_back_wheel_joint" type="continuous">
-    <axis xyz="0 1 0" />
-    <parent link="chassis"/>
-    <child link="right_back_wheel"/>
-    <origin rpy="0 0 0" xyz="-0.1 -0.08 0"/>
-  </joint> -->
 <gazebo>
   <plugin name="differential_drive_controller" filename="libgazebo_ros_diff_drive.so">

Commit message: some recognition wokring - need to redo cv for detection

File: urdf/robot.xacro (robot description, xacro)
@@ -133,5 +133,5 @@
   <link name="camera_link">
     <collision>
-      <origin xyz="0 0 0" rpy="0 0 0"/>
+      <origin xyz="0 0 0" rpy="1 0 0"/>
       <geometry>
     <box size="${camera_link} ${camera_link} ${camera_link}"/>

Commit message: Line Following Works! Changed Paramets for line follow Removed Delay in callback Moved robot wheels back

File: urdf/robot.xacro (robot description, xacro)
@@ -56,5 +56,5 @@
     <parent link="chassis"/>
     <child link="left_front_wheel"/>
-    <origin rpy="0 0 0" xyz="0.1 0.09 0"/>
+    <origin rpy="0 0 0" xyz="0.08 0.09 0"/>
   </joint>
   <link name="right_front_wheel">
@@ -78,5 +78,5 @@
     <parent link="chassis"/>
     <child link="right_front_wheel"/>
-    <origin rpy="0 0 0" xyz="0.1 -0.09 0"/>
+    <origin rpy="0 0 0" xyz="0.08 -0.09 0"/>
   </joint>
   <link name="left_back_wheel">
